Commit message: major finished wall, base c, and wall c

File: urdf/base_cabinet.urdf (robot description, URDF)
Before this commit: robot base_cabinet, 29 links, 28 joints
Links:
- added link base_cabinet_c1_door_handle_link, mass 0.09; collision mesh filename=package://clover_lab/meshes/handle.stl; visual mesh filename=package://clover_lab/meshes/handle.stl
- added link base_cabinet_c2_pull_out_handle_link, mass 0.09; collision mesh filename=package://clover_lab/meshes/handle.stl; visual mesh filename=package://clover_lab/meshes/handle.stl
- added link base_cabinet_c3_r1_drawer_handle_link, mass 0.09; collision mesh filename=package://clover_lab/meshes/handle.stl; visual mesh filename=package://clover_lab/meshes/handle.stl
- added link base_cabinet_c3_r2_drawer_handle_link, mass 0.09; collision mesh filename=package://clover_lab/meshes/handle.stl; visual mesh filename=package://clover_lab/meshes/handle.stl
- added link base_cabinet_c3_r3_drawer_handle_link, mass 0.09; collision mesh filename=package://clover_lab/meshes/handle.stl; visual mesh filename=package://clover_lab/meshes/handle.stl
- added link base_cabinet_c3_r4_drawer_handle_link, mass 0.09; collision mesh filename=package://clover_lab/meshes/handle.stl; visual mesh filename=package://clover_lab/meshes/handle.stl
- added link base_cabinet_c4_door_handle_link, mass 0.09; collision mesh filename=package://clover_lab/meshes/handle.stl; visual mesh filename=package://clover_lab/meshes/handle.stl
- added link base_cabinet_c5_door_handle_link, mass 0.09; collision mesh filename=package://clover_lab/meshes/handle.stl; visual mesh filename=package://clover_lab/meshes/handle.stl
Joints:
- added joint base_cabinet_c1_door_handle_joint: type fixed, parent base_cabinet_c1_door, child base_cabinet_c1_door_handle_link, origin xyz=0.008 0.35 0.28 rpy=1.5707963267948966 0 0
- added joint base_cabinet_c2_pull_out_handle_joint: type fixed, parent base_cabinet_c2_pull_out_front_panel, child base_cabinet_c2_pull_out_handle_link, origin xyz=0.008 0 0.34850000000000003 rpy=0 0 0
- added joint base_cabinet_c3_r1_drawer_handle_joint: type fixed, parent base_cabinet_c3_r1_drawer_front_panel, child base_cabinet_c3_r1_drawer_handle_link, origin xyz=0.008 0 0.048 rpy=0 0 0
- added joint base_cabinet_c3_r2_drawer_handle_joint: type fixed, parent base_cabinet_c3_r2_drawer_front_panel, child base_cabinet_c3_r2_drawer_handle_link, origin xyz=0.008 0 0.048 rpy=0 0 0
- added joint base_cabinet_c3_r3_drawer_handle_joint: type fixed, parent base_cabinet_c3_r3_drawer_front_panel, child base_cabinet_c3_r3_drawer_handle_link, origin xyz=0.008 0 0.048 rpy=0 0 0
- added joint base_cabinet_c3_r4_drawer_handle_joint: type fixed, parent base_cabinet_c3_r4_drawer_front_panel, child base_cabinet_c3_r4_drawer_handle_link, origin xyz=0.008 0 0.048 rpy=0 0 0
- added joint base_cabinet_c4_door_handle_joint: type fixed, parent base_cabinet_c4_door, child base_cabinet_c4_door_handle_link, origin xyz=0.008 0.35 0.28 rpy=1.5707963267948966 0 0
- added joint base_cabinet_c5_door_handle_joint: type fixed, parent base_cabinet_c5_door, child base_cabinet_c5_door_handle_link, origin xyz=0.008 -0.35 0.28 rpy=1.5707963267948966 0 0

File: urdf/clover_lab.urdf (robot description, URDF)
Before this commit: robot clover_lab, 37 links, 36 joints
Links:
- added link base_cabinet_c1_door_handle_link, mass 0.09; collision mesh filename=package://clover_lab/meshes/handle.stl; visual mesh filename=package://clover_lab/meshes/handle.stl
- added link base_cabinet_c2_pull_out_handle_link, mass 0.09; collision mesh filename=package://clover_lab/meshes/handle.stl; visual mesh filename=package://clover_lab/meshes/handle.stl
- added link base_cabinet_c3_r1_drawer_handle_link, mass 0.09; collision mesh filename=package://clover_lab/meshes/handle.stl; visual mesh filename=package://clover_lab/meshes/handle.stl
- added link base_cabinet_c3_r2_drawer_handle_link, mass 0.09; collision mesh filename=package://clover_lab/meshes/handle.stl; visual mesh filename=package://clover_lab/meshes/handle.stl
- added link base_cabinet_c3_r3_drawer_handle_link, mass 0.09; collision mesh filename=package://clover_lab/meshes/handle.stl; visual mesh filename=package://clover_lab/meshes/handle.stl
- added link base_cabinet_c3_r4_drawer_handle_link, mass 0.09; collision mesh filename=package://clover_lab/meshes/handle.stl; visual mesh filename=package://clover_lab/meshes/handle.stl
- added link base_cabinet_c4_door_handle_link, mass 0.09; collision mesh filename=package://clover_lab/meshes/handle.stl; visual mesh filename=package://clover_lab/meshes/handle.stl
- added link base_cabinet_c5_door_handle_link, mass 0.09; collision mesh filename=package://clover_lab/meshes/handle.stl; visual mesh filename=package://clover_lab/meshes/handle.stl
- added link lab_back_wall, mass 100; collision box size=0.1 3.2 2.7; visual box size=0.1 3.2 2.7
- added link lab_left_wall, mass 100; collision box size=6 0.1 2.7; visual box size=6 0.1 2.7
- added link wall_cabinet_c1_door_handle_link, mass 0.09; collision mesh filename=package://clover_lab/meshes/handle.stl; visual mesh filename=package://clover_lab/meshes/handle.stl
- added link wall_cabinet_c2_door_handle_link, mass 0.09; collision mesh filename=package://clover_lab/meshes/handle.stl; visual mesh filename=package://clover_lab/meshes/handle.stl
- link base_cabinet_c1_door: geometry collision box size=0.016 0.396 0.796; visual box size=0.016 0.396 0.796
- link base_cabinet_c4_door: geometry collision box size=0.016 0.396 0.796; visual box size=0.016 0.396 0.796
- link base_cabinet_c5_door: geometry collision box size=0.016 0.396 0.796; visual box size=0.016 0.396 0.796
Joints:
- added joint back_wall_joint: type fixed, parent world, child lab_back_wall, origin xyz=-3.05 0 1.35 rpy=0 0 0
- added joint base_cabinet_c1_door_handle_joint: type fixed, parent base_cabinet_c1_door, child base_cabinet_c1_door_handle_link, origin xyz=0.008 0.35 0.28 rpy=1.5707963267948966 0 0
- added joint base_cabinet_c2_pull_out_handle_joint: type fixed, parent base_cabinet_c2_pull_out_front_panel, child base_cabinet_c2_pull_out_handle_link, origin xyz=0.008 0 0.34850000000000003 rpy=0 0 0
- added joint base_cabinet_c3_r1_drawer_handle_joint: type fixed, parent base_cabinet_c3_r1_drawer_front_panel, child base_cabinet_c3_r1_drawer_handle_link, origin xyz=0.008 0 0.048 rpy=0 0 0
- added joint base_cabinet_c3_r2_drawer_handle_joint: type fixed, parent base_cabinet_c3_r2_drawer_front_panel, child base_cabinet_c3_r2_drawer_handle_link, origin xyz=0.008 0 0.048 rpy=0 0 0
- added joint base_cabinet_c3_r3_drawer_handle_joint: type fixed, parent base_cabinet_c3_r3_drawer_front_panel, child base_cabinet_c3_r3_drawer_handle_link, origin xyz=0.008 0 0.048 rpy=0 0 0
- added joint base_cabinet_c3_r4_drawer_handle_joint: type fixed, parent base_cabinet_c3_r4_drawer_front_panel, child base_cabinet_c3_r4_drawer_handle_link, origin xyz=0.008 0 0.048 rpy=0 0 0
- added joint base_cabinet_c4_door_handle_joint: type fixed, parent base_cabinet_c4_door, child base_cabinet_c4_door_handle_link, origin xyz=0.008 0.35 0.28 rpy=1.5707963267948966 0 0
- added joint base_cabinet_c5_door_handle_joint: type fixed, parent base_cabinet_c5_door, child base_cabinet_c5_door_handle_link, origin xyz=0.008 -0.35 0.28 rpy=1.5707963267948966 0 0
- added joint left_wall_joint: type fixed, parent world, child lab_left_wall, origin xyz=0 1.6500000000000001 1.35 rpy=0 0 0
- added joint wall_cabinet_c1_door_handle_joint: type fixed, parent wall_cabinet_c1_door, child wall_cabinet_c1_door_handle_link, origin xyz=0.008 0.48 -0.35 rpy=0 0 0
- added joint wall_cabinet_c2_door_handle_joint: type fixed, parent wall_cabinet_c2_door, child wall_cabinet_c2_door_handle_link, origin xyz=0.008 -0.28 -0.35 rpy=0 0 0
- joint wall_cabinet_reference: origin xyz=-2.7 0.4 2.045 rpy=0 0 0 -> xyz=-3.0 0.4 2.045 rpy=0 0 0

File: urdf/wall_cabinet.urdf (robot description, URDF)
Before this commit: robot wall_cabinet, 7 links, 6 joints
Links:
- added link wall_cabinet_c1_door_handle_link, mass 0.09; collision mesh filename=package://clover_lab/meshes/handle.stl; visual mesh filename=package://clover_lab/meshes/handle.stl
- added link wall_cabinet_c2_door_handle_link, mass 0.09; collision mesh filename=package://clover_lab/meshes/handle.stl; visual mesh filename=package://clover_lab/meshes/handle.stl
Joints:
- added joint wall_cabinet_c1_door_handle_joint: type fixed, parent wall_cabinet_c1_door, child wall_cabinet_c1_door_handle_link, origin xyz=0.008 0.48 -0.35 rpy=0 0 0
- added joint wall_cabinet_c2_door_handle_joint: type fixed, parent wall_cabinet_c2_door, child wall_cabinet_c2_door_handle_link, origin xyz=0.008 -0.28 -0.35 rpy=0 0 0

File: xacro/base_cabinet.urdf.xacro (robot description, xacro)
@@ -7,5 +7,7 @@
   <xacro:arg name="simulator" default="none"/>
   <xacro:property name="simulator" value="$(arg simulator)"/>
-  <xacro:include filename="components.xacro"/>
+  <xacro:include filename="include/materials.xacro"/>
+  <xacro:include filename="include/properties.xacro"/>
+  <xacro:include filename="include/components.xacro"/>
   <xacro:include filename="base_cabinet.xacro"/>
   <xacro:if value="${simulator == 'mujoco'}">

File: xacro/base_cabinet.xacro (robot description, xacro)
@@ -1,63 +1,4 @@
 <?xml version="1.0"?>
 <robot name="base_cabinet" xmlns:xacro="http://wiki.ros.org/xacro">
-  <!-- Using meter, kg -->
-  <xacro:property name="base_xdim" value="0.6"/>
-  <xacro:property name="base_ydim" value="1.8"/>
-  <xacro:property name="base_zdim" value="0.08"/>
-  <xacro:property name="base_mass" value="20"/>
-  <!-- Frame refers to the main part of the cabinet -->
-  <xacro:property name="bc_frame_xdim" value="0.6"/>
-  <xacro:property name="bc_frame_ydim" value="1.8"/>
-  <xacro:property name="bc_frame_zdim" value="0.8"/>
-  <xacro:property name="column_ydim" value="0.4"/>
-  <xacro:property name="row_zdim" value="${bc_frame_zdim/4}"/>
-  <xacro:property name="thickness" value="0.016"/>
-  <xacro:property name="tolerance" value="0.004"/>
-  <xacro:property name="bc_frame_back_panel_xdim" value="${thickness}"/>
-  <xacro:property name="bc_frame_back_panel_ydim" value="${bc_frame_ydim}"/>
-  <xacro:property name="bc_frame_back_panel_zdim" value="${bc_frame_zdim}"/>
-  <xacro:property name="bc_frame_back_panel_mass" value="20"/>
-  <xacro:property name="bc_frame_side_panel_xdim" value="${bc_frame_xdim}"/>
-  <xacro:property name="bc_frame_side_panel_ydim" value="${thickness}"/>
-  <xacro:property name="bc_frame_side_panel_zdim" value="${bc_frame_zdim}"/>
-  <xacro:property name="bc_frame_side_panel_mass" value="5"/>
-  <!-- https://www.ikea.com.hk/zh/products/kitchen-worktops/kitchen-worktops/lilltrask-art-40280659-->
-  <xacro:property name="worktop_xdim" value="0.635"/>
-  <xacro:property name="worktop_ydim" value="1.86"/>
-  <xacro:property name="worktop_zdim" value="0.028"/>
-  <xacro:property name="worktop_mass" value="20.65"/>
-  <!-- https://www.ikea.com.hk/en/products/kitchen-fronts/kitchen-fronts-cover-panels-and-plinth/enhet-art-90481556 -->
-  <xacro:property name="door_xdim" value="${thickness}"/>
-  <xacro:property name="door_ydim" value="${column_ydim-tolerance}"/>
-  <xacro:property name="door_zdim" value="${bc_frame_zdim-tolerance}"/>
-  <xacro:property name="door_mass" value="3.31"/>
-  <!-- https://www.ikea.com.hk/en/products/kitchen-fronts/kitchen-fronts-cover-panels-and-plinth/enhet-art-30481559 -->
-  <xacro:property name="drawer_front_panel_xdim" value="${thickness}"/>
-  <xacro:property name="drawer_front_panel_ydim" value="${column_ydim-tolerance}"/>
-  <xacro:property name="drawer_front_panel_zdim" value="${row_zdim-tolerance}"/>
-  <xacro:property name="drawer_front_panel_mass" value="0.75"/>
-  <!-- Drawer interior, bc_frame size: X60cm Y40cm Z20cm -->
-  <!-- https://www.ikea.com.hk/en/products/kitchen-fixed-interiors/kitchen-fixed-interiors/maximera-art-70271111-->
-  <xacro:property name="drawer_interior_xdim" value="0.542"/>
-  <xacro:property name="drawer_interior_ydim" value="0.364"/>
-  <xacro:property name="drawer_interior_zdim" value="0.144"/>
-  <xacro:property name="drawer_side_panel_xdim" value="${drawer_interior_xdim}"/>
-  <xacro:property name="drawer_side_panel_ydim" value="${thickness}"/>
-  <xacro:property name="drawer_side_panel_zdim" value="${drawer_interior_zdim}"/>
-  <xacro:property name="drawer_side_panel_mass" value="2"/>
-  <xacro:property name="drawer_bottom_panel_xdim" value="${drawer_interior_xdim}"/>
-  <xacro:property name="drawer_bottom_panel_ydim" value="${drawer_interior_ydim}"/>
-  <xacro:property name="drawer_bottom_panel_zdim" value="${thickness}"/>
-  <xacro:property name="drawer_bottom_panel_mass" value="3"/>
-  <xacro:property name="drawer_back_panel_xdim" value="${thickness}"/>
-  <xacro:property name="drawer_back_panel_ydim" value="${drawer_interior_ydim}"/>
-  <xacro:property name="drawer_back_panel_zdim" value="${drawer_interior_zdim}"/>
-  <xacro:property name="drawer_back_panel_mass" value="2"/>
-  <!-- https://www.ikea.com.hk/en/products/kitchen-fronts/kitchen-fronts-cover-panels-and-plinth/askersund-art-50331776-->
-  <xacro:property name="pull_out_front_panel_xdim" value="${thickness}"/>
-  <xacro:property name="pull_out_front_panel_ydim" value="0.197"/>
-  <xacro:property name="pull_out_front_panel_zdim" value="0.797"/>
-  <xacro:property name="pull_out_front_panel_mass" value="1.66"/>
-  <!-- https://www.ikea.com.hk/en/products/kitchen-fixed-interiors/kitchen-fixed-interiors/maximera-art-80297276-->
   <xacro:macro name="drawer" params="prefix name parent xyz">
     <xacro:box_link prefix="${prefix}" link_name="${name}_front_panel" mass="${drawer_front_panel_mass}"
@@ -73,4 +14,6 @@
       <axis xyz="1 0 0"/>
     </joint>
+    <xacro:handle prefix="${prefix}" name="${name}" parent="${prefix}_${name}_front_panel"
+                  xyz="${drawer_front_panel_xdim/2} 0 ${drawer_front_panel_zdim/2-0.05}"/>
     <xacro:box_link prefix="${prefix}" link_name="${name}_bottom_panel" mass="${drawer_bottom_panel_mass}"
                     xdim="${drawer_bottom_panel_xdim}" ydim="${drawer_bottom_panel_ydim}"
@@ -128,4 +71,6 @@
       <axis xyz="1 0 0"/>
     </joint>
+    <xacro:handle prefix="${prefix}" name="${name}" parent="${prefix}_${name}_front_panel"
+                  xyz="${pull_out_front_panel_xdim/2} 0 ${pull_out_front_panel_zdim/2-0.05}"/>
     <!--    <xacro:box_link prefix="${prefix}" link_name="${name}_bottom_panel" mass="${drawer_bottom_panel_mass}"-->
     <!--                    xdim="${drawer_bottom_panel_xdim}" ydim="${drawer_bottom_panel_ydim}"-->
@@ -162,6 +107,6 @@
   <!-- Assembles -->
   <xacro:macro name="bc_frame">
-    <xacro:box_link prefix="bc_frame" link_name="base_link" mass="${base_mass}" xdim="${base_xdim}" ydim="${base_ydim}"
-                    zdim="${base_zdim}" material="White"/>
+    <xacro:box_link prefix="bc_frame" link_name="base_link" mass="${bc_base_mass}" xdim="${bc_base_xdim}" ydim="${bc_base_ydim}"
+                    zdim="${bc_base_zdim}" material="White"/>
     <xacro:box_link prefix="bc_frame" link_name="left_side_panel" mass="${bc_frame_side_panel_mass}"
                     xdim="${bc_frame_side_panel_xdim}" ydim="${bc_frame_side_panel_ydim}"
@@ -169,5 +114,5 @@
                     material="White"/>
     <joint name="bc_frame_left_side_panel_joint" type="fixed">
-      <origin xyz="0 ${(base_ydim-bc_frame_side_panel_ydim)/2} ${(base_zdim+bc_frame_side_panel_zdim)/2}" rpy="0 0 0"/>
+      <origin xyz="0 ${(bc_base_ydim-bc_frame_side_panel_ydim)/2} ${(bc_base_zdim+bc_frame_side_panel_zdim)/2}" rpy="0 0 0"/>
       <parent link="bc_frame_base_link"/>
       <child link="bc_frame_left_side_panel"/>
@@ -178,5 +123,5 @@
                     material="White"/>
     <joint name="bc_frame_right_side_panel_joint" type="fixed">
-      <origin xyz="0 ${(-base_ydim+bc_frame_side_panel_ydim)/2} ${(base_zdim+bc_frame_side_panel_zdim)/2}" rpy="0 0 0"/>
+      <origin xyz="0 ${(-bc_base_ydim+bc_frame_side_panel_ydim)/2} ${(bc_base_zdim+bc_frame_side_panel_zdim)/2}" rpy="0 0 0"/>
       <parent link="bc_frame_base_link"/>
       <child link="bc_frame_right_side_panel"/>
@@ -187,5 +132,5 @@
                     material="White"/>
     <joint name="bc_frame_back_panel_joint" type="fixed">
-      <origin xyz="${(-base_xdim+bc_frame_back_panel_xdim)/2} 0 ${(base_zdim+bc_frame_back_panel_zdim)/2}" rpy="0 0 0"/>
+      <origin xyz="${(-bc_base_xdim+bc_frame_back_panel_xdim)/2} 0 ${(bc_base_zdim+bc_frame_back_panel_zdim)/2}" rpy="0 0 0"/>
       <parent link="bc_frame_base_link"/>
       <child link="bc_frame_back_panel"/>
@@ -195,5 +140,5 @@
                     material="White"/>
     <joint name="bc_frame_worktop_joint" type="fixed">
-      <origin xyz="0 0 ${(base_zdim+worktop_zdim)/2+bc_frame_back_panel_zdim}" rpy="0 0 0"/>
+      <origin xyz="0 0 ${(bc_base_zdim+worktop_zdim)/2+bc_frame_back_panel_zdim}" rpy="0 0 0"/>
       <parent link="bc_frame_base_link"/>
       <child link="bc_frame_worktop"/>
@@ -212,34 +157,34 @@
     <!-- Rightmost 1st column -->
     <xacro:door prefix="${prefix}" name="c1_door" parent="bc_frame_base_link"
-                xyz="${base_xdim/2} ${-base_ydim/2+bc_frame_side_panel_ydim} ${(base_zdim+bc_frame_side_panel_zdim)/2}"
-                mass="${door_mass}" xdim="${door_xdim}" ydim="${door_ydim}" zdim="${door_zdim}"
-                hinge="right"/>
+                xyz="${bc_base_xdim/2} ${-bc_base_ydim/2+bc_frame_side_panel_ydim} ${(bc_base_zdim+bc_frame_side_panel_zdim)/2}"
+                mass="${bc_door_mass}" xdim="${bc_door_xdim}" ydim="${bc_door_ydim}" zdim="${bc_door_zdim}"
+                hinge="right" handle_xyz="0.008 0.35 0.28" handle_rpy="${M_PI/2} 0 0"/>
     <!-- Rightmost 2nd column -->
     <xacro:pull_out prefix="${prefix}" name="c2_pull_out" parent="bc_frame_base_link"
-                    xyz="${(base_xdim+thickness)/2} ${base_ydim/2-bc_frame_side_panel_ydim-column_ydim*3.25}
-                       ${(base_zdim+bc_frame_zdim)/2}"/>
+                    xyz="${(bc_base_xdim+thickness)/2} ${bc_base_ydim/2-bc_frame_side_panel_ydim-bc_column_ydim*3.25}
+                       ${(bc_base_zdim+bc_frame_zdim)/2}"/>
     <!-- Rightmost 3rd column -->
     <xacro:drawer prefix="${prefix}" name="c3_r1_drawer" parent="bc_frame_base_link"
-                  xyz="${(base_xdim+drawer_front_panel_xdim)/2} ${base_ydim/2-bc_frame_side_panel_ydim-column_ydim*2.5}
-                     ${(base_zdim-row_zdim)/2+bc_frame_zdim}"/>
+                  xyz="${(bc_base_xdim+drawer_front_panel_xdim)/2} ${bc_base_ydim/2-bc_frame_side_panel_ydim-bc_column_ydim*2.5}
+                     ${(bc_base_zdim-bc_row_zdim)/2+bc_frame_zdim}"/>
     <xacro:drawer prefix="${prefix}" name="c3_r2_drawer" parent="bc_frame_base_link"
-                  xyz="${(base_xdim+drawer_front_panel_xdim)/2} ${base_ydim/2-bc_frame_side_panel_ydim-column_ydim*2.5}
-                     ${(base_zdim-row_zdim*3)/2+bc_frame_zdim}"/>
+                  xyz="${(bc_base_xdim+drawer_front_panel_xdim)/2} ${bc_base_ydim/2-bc_frame_side_panel_ydim-bc_column_ydim*2.5}
+                     ${(bc_base_zdim-bc_row_zdim*3)/2+bc_frame_zdim}"/>
     <xacro:drawer prefix="${prefix}" name="c3_r3_drawer" parent="bc_frame_base_link"
-                  xyz="${(base_xdim+drawer_front_panel_xdim)/2} ${base_ydim/2-bc_frame_side_panel_ydim-column_ydim*2.5}
-                     ${(base_zdim-row_zdim*5)/2+bc_frame_zdim}"/>
+                  xyz="${(bc_base_xdim+drawer_front_panel_xdim)/2} ${bc_base_ydim/2-bc_frame_side_panel_ydim-bc_column_ydim*2.5}
+                     ${(bc_base_zdim-bc_row_zdim*5)/2+bc_frame_zdim}"/>
     <xacro:drawer prefix="${prefix}" name="c3_r4_drawer" parent="bc_frame_base_link"
-                  xyz="${(base_xdim+drawer_front_panel_xdim)/2} ${base_ydim/2-bc_frame_side_panel_ydim-column_ydim*2.5}
-                     ${(base_zdim-row_zdim*7)/2+bc_frame_zdim}"/>
+                  xyz="${(bc_base_xdim+drawer_front_panel_xdim)/2} ${bc_base_ydim/2-bc_frame_side_panel_ydim-bc_column_ydim*2.5}
+                     ${(bc_base_zdim-bc_row_zdim*7)/2+bc_frame_zdim}"/>
     <!-- Rightmost 4th column -->
     <xacro:door prefix="${prefix}" name="c4_door" parent="bc_frame_base_link"
-                xyz="${base_xdim/2} ${base_ydim/2-bc_frame_side_panel_ydim-column_ydim*2} ${(base_zdim+bc_frame_side_panel_zdim)/2}"
-                mass="${door_mass}" xdim="${door_xdim}" ydim="${door_ydim}" zdim="${door_zdim}"
-                hinge="right"/>
+                xyz="${bc_base_xdim/2} ${bc_base_ydim/2-bc_frame_side_panel_ydim-bc_column_ydim*2} ${(bc_base_zdim+bc_frame_side_panel_zdim)/2}"
+                mass="${bc_door_mass}" xdim="${bc_door_xdim}" ydim="${bc_door_ydim}" zdim="${bc_door_zdim}"
+                hinge="right" handle_xyz="0.008 0.35 0.28" handle_rpy="${M_PI/2} 0 0"/>
     <!-- Rightmost 5th column -->
     <xacro:door prefix="${prefix}" name="c5_door" parent="bc_frame_base_link"
-                xyz="${base_xdim/2} ${base_ydim/2-bc_frame_side_panel_ydim} ${(base_zdim+bc_frame_side_panel_zdim)/2}"
-                mass="${door_mass}" xdim="${door_xdim}" ydim="${door_ydim}" zdim="${door_zdim}"
-                hinge="left"/>
+                xyz="${bc_base_xdim/2} ${bc_base_ydim/2-bc_frame_side_panel_ydim} ${(bc_base_zdim+bc_frame_side_panel_zdim)/2}"
+                mass="${bc_door_mass}" xdim="${bc_door_xdim}" ydim="${bc_door_ydim}" zdim="${bc_door_zdim}"
+                hinge="left" handle_xyz="0.008 -0.35 0.28" handle_rpy="${M_PI/2} 0 0"/>
   </xacro:macro>
 </robot>

File: xacro/clover_lab.urdf.xacro (robot description, xacro)
@@ -5,5 +5,8 @@
   <xacro:arg name="simulator" default="none"/>
   <xacro:property name="simulator" value="$(arg simulator)"/>
-  <xacro:include filename="components.xacro"/>
+  <xacro:include filename="include/materials.xacro"/>
+  <xacro:include filename="include/properties.xacro"/>
+  <xacro:include filename="include/components.xacro"/>
+  <xacro:include filename="include/wall.xacro"/>
   <xacro:include filename="base_cabinet.xacro"/>
   <xacro:include filename="wall_cabinet.xacro"/>
@@ -19,13 +22,14 @@
     <link name="world"/>
     <joint name="base_cabinet_reference" type="fixed">
-      <origin xyz="-2.7 0.2 ${base_zdim/2}" rpy="0 0 0"/>
+      <origin xyz="-2.7 0.2 ${bc_base_zdim/2}" rpy="0 0 0"/>
       <parent link="world"/>
       <child link="bc_frame_base_link"/>
     </joint>
     <joint name="wall_cabinet_reference" type="fixed">
-      <origin xyz="-2.7 0.4 ${1.64+0.81/2}" rpy="0 0 0"/>
+      <origin xyz="${-space_xdim/2} 0.4 ${1.64+wc_frame_zdim/2}" rpy="0 0 0"/>
       <parent link="world"/>
       <child link="wc_frame_back_panel"/>
     </joint>
   </xacro:unless>
+  <xacro:wall/>
 </robot>
