Commit message: major finished wall, base c, and wall c

File: xacro/include/components.xacro (robot description, xacro)
@@ -1,5 +1,4 @@
 <?xml version="1.0"?>
 <robot name="components" xmlns:xacro="http://wiki.ros.org/xacro">
-  <xacro:include filename="materials.xacro"/>
   <xacro:property name="M_PI" value="3.1415926535897931"/>
   <!-- https://www.ikea.com.hk/en/products/knobs-and-handles/knobs-and-handles/bagganas-art-70338423 -->
@@ -56,33 +55,34 @@
     </link>
   </xacro:macro>
-  <!--  <xacro:macro name="handle" params="prefix parent *origin">-->
-  <!--    <link name="${prefix}_handle">-->
-  <!--      <visual>-->
-  <!--        <origin xyz="0 0 0" rpy="0 0 0"/>-->
-  <!--        &lt;!&ndash;        <geometry>&ndash;&gt;-->
-  <!--        &lt;!&ndash;          <box size="${worktop_ydim worktop_xdim worktop_zdim}"/>&ndash;&gt;-->
-  <!--        &lt;!&ndash;        </geometry>&ndash;&gt;-->
-  <!--        <material name="Black"/>-->
-  <!--      </visual>-->
-  <!--      <collision>-->
-  <!--        <origin xyz="0 0 0" rpy="0 0 0"/>-->
-  <!--        &lt;!&ndash;        <geometry>&ndash;&gt;-->
-  <!--        &lt;!&ndash;          <box size="${worktop_ydim worktop_xdim worktop_zdim}"/>&ndash;&gt;-->
-  <!--        &lt;!&ndash;        </geometry>&ndash;&gt;-->
-  <!--      </collision>-->
-  <!--      <inertial>-->
-  <!--        <mass value="${handle_mass}"/>-->
-  <!--        &lt;!&ndash;        <origin xyz="0 0 0"/>&ndash;&gt;-->
-  <!--        &lt;!&ndash;        <xacro:box_inertia mass="${worktop_mass}" ydim="${worktop_ydim}" xdim="${worktop_xdim}"&ndash;&gt;-->
-  <!--        &lt;!&ndash;                           zdim="${worktop_zdim}"/>&ndash;&gt;-->
-  <!--      </inertial>-->
-  <!--    </link>-->
-  <!--    <joint name="{prefix}_handle_joint" type="fixed">-->
-  <!--      <parent link="${parent}"/>-->
-  <!--      <child link="{prefix}_handle_link"/>-->
-  <!--      <xacro:insert_block name="origin"/>-->
-  <!--    </joint>-->
-  <!--  </xacro:macro>-->
-  <xacro:macro name="door" params="prefix name parent xyz mass xdim ydim zdim hinge">
+  <xacro:macro name="handle" params="prefix name parent xyz rpy:='0 0 0'">
+    <link name="${prefix}_${name}_handle_link">
+      <visual>
+        <origin xyz="0 0 0" rpy="0 0 0"/>
+        <geometry>
+          <mesh filename="package://clover_lab/meshes/handle.stl"/>
+        </geometry>
+        <material name="Black"/>
+      </visual>
+      <collision>
+        <origin xyz="0 0 0" rpy="0 0 0"/>
+        <geometry>
+          <mesh filename="package://clover_lab/meshes/handle.stl"/>
+        </geometry>
+      </collision>
+      <inertial>
+        <mass value="${handle_mass}"/>
+        <origin xyz="0 0 0"/>
+        <inertia ixx="${211.711 * 1e-6}" ixy="0" ixz="0"
+                 iyy="${63.764 * 1e-6}" iyz="0"
+                 izz="${274.426 * 1e-6}"/>
+      </inertial>
+    </link>
+    <joint name="${prefix}_${name}_handle_joint" type="fixed">
+      <parent link="${parent}"/>
+      <child link="${prefix}_${name}_handle_link"/>
+      <origin xyz="${xyz}" rpy="${rpy}"/>
+    </joint>
+  </xacro:macro>
+  <xacro:macro name="door" params="prefix name parent xyz mass xdim ydim zdim hinge handle_xyz handle_rpy">
     <xacro:box_link prefix="${prefix}" link_name="${name}" mass="${mass}"
                     xdim="${xdim}" ydim="${ydim}" zdim="${zdim}"
@@ -101,4 +101,5 @@
       </xacro:unless>
     </joint>
+    <xacro:handle prefix="${prefix}" name="${name}" parent="${prefix}_${name}" xyz="${handle_xyz}" rpy="${handle_rpy}"/>
   </xacro:macro>
 </robot>

File: xacro/include/materials.xacro (robot description, xacro)
@@ -13,3 +13,6 @@
     <color rgba="0.89 0.81 0.69 1.0"/>
   </material>
+  <material name="Green">
+    <color rgba="0.8 1 0.8 1.0"/>
+  </material>
 </robot>

File: xacro/wall_cabinet.urdf.xacro (robot description, xacro)
@@ -7,5 +7,7 @@
   <xacro:arg name="simulator" default="none"/>
   <xacro:property name="simulator" value="$(arg simulator)"/>
-  <xacro:include filename="components.xacro"/>
+  <xacro:include filename="include/materials.xacro"/>
+  <xacro:include filename="include/properties.xacro"/>
+  <xacro:include filename="include/components.xacro"/>
   <xacro:include filename="wall_cabinet.xacro"/>
   <xacro:if value="${simulator == 'mujoco'}">

File: xacro/wall_cabinet.xacro (robot description, xacro)
@@ -1,28 +1,4 @@
 <?xml version="1.0"?>
 <robot name="wall_cabinet" xmlns:xacro="http://wiki.ros.org/xacro">
-  <!-- Using meter, kg -->
-  <!-- Frame refers to the main part of the cabinet -->
-  <xacro:property name="wc_frame_xdim" value="0.39"/>
-  <xacro:property name="wc_frame_ydim" value="1"/>
-  <xacro:property name="wc_frame_zdim" value="0.81"/>
-  <xacro:property name="thickness" value="0.016"/>
-  <xacro:property name="tolerance" value="0.004"/>
-  <!-- https://www.ikea.com.hk/en/products/kitchen-cabinets-and-worktops/kitchen-cabinets/enhet-spr-49395118 -->
-  <xacro:property name="wc_frame_h_panel_xdim" value="${wc_frame_xdim-thickness}"/>
-  <xacro:property name="wc_frame_h_panel_ydim" value="${wc_frame_ydim}"/>
-  <xacro:property name="wc_frame_h_panel_zdim" value="${thickness}"/>
-  <xacro:property name="wc_frame_h_panel_mass" value="20"/>
-  <xacro:property name="wc_frame_side_panel_xdim" value="${wc_frame_xdim-thickness}"/>
-  <xacro:property name="wc_frame_side_panel_ydim" value="${thickness}"/>
-  <xacro:property name="wc_frame_side_panel_zdim" value="${wc_frame_zdim}"/>
-  <xacro:property name="wc_frame_side_panel_mass" value="10"/>
-  <xacro:property name="wc_frame_back_panel_xdim" value="${thickness}"/>
-  <xacro:property name="wc_frame_back_panel_ydim" value="${wc_frame_ydim}"/>
-  <xacro:property name="wc_frame_back_panel_zdim" value="${wc_frame_zdim}"/>
-  <xacro:property name="wc_frame_back_panel_mass" value="20"/>
-  <!-- https://www.ikea.com.hk/en/products/kitchen-fronts/kitchen-fronts-cover-panels-and-plinth/enhet-art-90481556 -->
-  <xacro:property name="door_xdim" value="${thickness}"/>
-  <xacro:property name="door_zdim" value="${wc_frame_zdim-tolerance}"/>
-  <xacro:property name="door_mass" value="3.31"/>
   <!-- Assembles -->
   <xacro:macro name="wc_frame">
@@ -79,12 +55,12 @@
     <!-- Rightmost 1st column -->
     <xacro:door prefix="${prefix}" name="c1_door" parent="wc_frame_back_panel"
-                xyz="${wc_frame_side_panel_xdim-door_xdim/2} ${-wc_frame_back_panel_ydim/2} 0"
-                mass="${door_mass}" xdim="${door_xdim}" ydim="${0.6-tolerance}" zdim="${door_zdim}"
-                hinge="right"/>
+                xyz="${wc_frame_side_panel_xdim-wc_door_xdim/2} ${-wc_frame_back_panel_ydim/2} 0"
+                mass="${door_mass}" xdim="${wc_door_xdim}" ydim="${0.6-tolerance}" zdim="${wc_door_zdim}"
+                hinge="right" handle_xyz="0.008 0.48 -0.35" handle_rpy="0 0 0"/>
     <!-- Rightmost 2nd column -->
     <xacro:door prefix="${prefix}" name="c2_door" parent="wc_frame_back_panel"
-                xyz="${wc_frame_side_panel_xdim-door_xdim/2} ${wc_frame_back_panel_ydim/2} 0"
-                mass="${door_mass}" xdim="${door_xdim}" ydim="${0.4-tolerance}" zdim="${door_zdim}"
-                hinge="left"/>
+                xyz="${wc_frame_side_panel_xdim-wc_door_xdim/2} ${wc_frame_back_panel_ydim/2} 0"
+                mass="${door_mass}" xdim="${wc_door_xdim}" ydim="${0.4-tolerance}" zdim="${wc_door_zdim}"
+                hinge="left" handle_xyz="0.008 -0.28 -0.35" handle_rpy="0 0 0"/>
   </xacro:macro>
 </robot>
