Commit message: add interior shelf

File: urdf/base_cabinet.urdf (robot description, URDF)
Before this commit: robot base_cabinet, 37 links, 36 joints
Links:
- added link bc_frame_c1_v_shelf, mass 10; collision box size=0.6 0.04 0.8; visual box size=0.6 0.04 0.8
- added link bc_frame_c2_v_shelf, mass 10; collision box size=0.6 0.04 0.8; visual box size=0.6 0.04 0.8
- added link bc_frame_c3_v_shelf, mass 10; collision box size=0.6 0.04 0.8; visual box size=0.6 0.04 0.8
- added link bc_frame_h1_shelf, mass 10; collision box size=0.6 0.8 0.02; visual box size=0.6 0.8 0.02
- added link bc_frame_h2_shelf, mass 10; collision box size=0.6 0.8 0.02; visual box size=0.6 0.8 0.02
- link base_cabinet_c2_pull_out_front_panel: geometry collision box size=0.016 0.196 0.796; visual box size=0.016 0.196 0.796
- link base_cabinet_c3_r1_drawer_back_panel: geometry collision box size=0.016 0.35 0.144; visual box size=0.016 0.35 0.144
- link base_cabinet_c3_r1_drawer_bottom_panel: geometry collision box size=0.542 0.35 0.016; visual box size=0.542 0.35 0.016
- link base_cabinet_c3_r2_drawer_back_panel: geometry collision box size=0.016 0.35 0.144; visual box size=0.016 0.35 0.144
- link base_cabinet_c3_r2_drawer_bottom_panel: geometry collision box size=0.542 0.35 0.016; visual box size=0.542 0.35 0.016
- link base_cabinet_c3_r3_drawer_back_panel: geometry collision box size=0.016 0.35 0.144; visual box size=0.016 0.35 0.144
- link base_cabinet_c3_r3_drawer_bottom_panel: geometry collision box size=0.542 0.35 0.016; visual box size=0.542 0.35 0.016
- link base_cabinet_c3_r4_drawer_back_panel: geometry collision box size=0.016 0.35 0.144; visual box size=0.016 0.35 0.144
- link base_cabinet_c3_r4_drawer_bottom_panel: geometry collision box size=0.542 0.35 0.016; visual box size=0.542 0.35 0.016
- link bc_frame_base_link: geometry collision box size=0.6 1.8 0.12; visual box size=0.6 1.8 0.12
Joints:
- added joint bc_frame_c1_v_shelf_joint: type fixed, parent bc_frame_base_link, child bc_frame_c1_v_shelf, origin xyz=0 -0.5 0.46
- added joint bc_frame_c2_v_shelf_joint: type fixed, parent bc_frame_base_link, child bc_frame_c2_v_shelf, origin xyz=0 -0.29999999999999993 0.46
- added joint bc_frame_c3_v_shelf_joint: type fixed, parent bc_frame_base_link, child bc_frame_c3_v_shelf, origin xyz=0 0.09999999999999998 0.46
- added joint bc_frame_h1_shelf_joint: type fixed, parent bc_frame_base_link, child bc_frame_h1_shelf, origin xyz=0 0.5000000000000001 0.6100000000000001
- added joint bc_frame_h2_shelf_joint: type fixed, parent bc_frame_base_link, child bc_frame_h2_shelf, origin xyz=0 0.5000000000000001 0.39000000000000007
- joint base_cabinet_c1_door_joint: origin xyz=0.3 -0.884 0.44 -> xyz=0.308 -0.9 0.46
- joint base_cabinet_c2_pull_out_front_panel_joint: origin xyz=0.308 -0.41600000000000004                        0.44 -> xyz=0.308                          -0.4                          0.46
- joint base_cabinet_c2_pull_out_handle_joint: origin xyz=0.008 0 0.34850000000000003 rpy=0 0 0 -> xyz=0.008 0 0.34800000000000003 rpy=0 0 0
- joint base_cabinet_c3_r1_drawer_front_panel_joint: origin xyz=0.308 -0.11599999999999999                      0.74 -> xyz=0.308                        -0.09999999999999998                        0.76
- joint base_cabinet_c3_r2_drawer_front_panel_joint: origin xyz=0.308 -0.11599999999999999                      0.54 -> xyz=0.308                        -0.09999999999999998                        0.56
- joint base_cabinet_c3_r3_drawer_front_panel_joint: origin xyz=0.308 -0.11599999999999999                      0.34 -> xyz=0.308                        -0.09999999999999998                        0.36000000000000004
- joint base_cabinet_c3_r4_drawer_front_panel_joint: origin xyz=0.308 -0.11599999999999999                      0.14 -> xyz=0.308                        -0.09999999999999998                        0.15999999999999992
- joint base_cabinet_c4_door_joint: origin xyz=0.3 0.08399999999999996 0.44 -> xyz=0.308                      0.09999999999999998                      0.46
- joint base_cabinet_c5_door_joint: origin xyz=0.3 0.884 0.44 -> xyz=0.308                      0.9                      0.46
- joint bc_frame_back_panel_joint: origin xyz=-0.292 0 0.44 rpy=0 0 0 -> xyz=-0.292 0 0.46 rpy=0 0 0
- joint bc_frame_left_side_panel_joint: origin xyz=0 0.892 0.44 rpy=0 0 0 -> xyz=0 0.892 0.46 rpy=0 0 0
- joint bc_frame_right_side_panel_joint: origin xyz=0 -0.892 0.44 rpy=0 0 0 -> xyz=0 -0.892 0.46 rpy=0 0 0
- joint bc_frame_worktop_joint: origin xyz=0 0 0.8540000000000001 rpy=0 0 0 -> xyz=0 0 0.874

File: urdf/clover_lab.urdf (robot description, URDF)
Before this commit: robot clover_lab, 49 links, 48 joints
Links:
- added link bc_frame_c1_v_shelf, mass 10; collision box size=0.6 0.04 0.8; visual box size=0.6 0.04 0.8
- added link bc_frame_c2_v_shelf, mass 10; collision box size=0.6 0.04 0.8; visual box size=0.6 0.04 0.8
- added link bc_frame_c3_v_shelf, mass 10; collision box size=0.6 0.04 0.8; visual box size=0.6 0.04 0.8
- added link bc_frame_h1_shelf, mass 10; collision box size=0.6 0.8 0.02; visual box size=0.6 0.8 0.02
- added link bc_frame_h2_shelf, mass 10; collision box size=0.6 0.8 0.02; visual box size=0.6 0.8 0.02
- added link wc_frame_c1_v_shelf, mass 10; collision box size=0.39 0.04 0.81; visual box size=0.39 0.04 0.81
- added link wc_frame_h1_shelf, mass 10; collision box size=0.39 1 0.02; visual box size=0.39 1 0.02
- added link wc_frame_h2_shelf, mass 10; collision box size=0.39 1 0.02; visual box size=0.39 1 0.02
- link base_cabinet_c2_pull_out_front_panel: geometry collision box size=0.016 0.196 0.796; visual box size=0.016 0.196 0.796
- link base_cabinet_c3_r1_drawer_back_panel: geometry collision box size=0.016 0.35 0.144; visual box size=0.016 0.35 0.144
- link base_cabinet_c3_r1_drawer_bottom_panel: geometry collision box size=0.542 0.35 0.016; visual box size=0.542 0.35 0.016
- link base_cabinet_c3_r2_drawer_back_panel: geometry collision box size=0.016 0.35 0.144; visual box size=0.016 0.35 0.144
- link base_cabinet_c3_r2_drawer_bottom_panel: geometry collision box size=0.542 0.35 0.016; visual box size=0.542 0.35 0.016
- link base_cabinet_c3_r3_drawer_back_panel: geometry collision box size=0.016 0.35 0.144; visual box size=0.016 0.35 0.144
- link base_cabinet_c3_r3_drawer_bottom_panel: geometry collision box size=0.542 0.35 0.016; visual box size=0.542 0.35 0.016
- link base_cabinet_c3_r4_drawer_back_panel: geometry collision box size=0.016 0.35 0.144; visual box size=0.016 0.35 0.144
- link base_cabinet_c3_r4_drawer_bottom_panel: geometry collision box size=0.542 0.35 0.016; visual box size=0.542 0.35 0.016
- link bc_frame_base_link: geometry collision box size=0.6 1.8 0.12; visual box size=0.6 1.8 0.12
- link wc_frame_bottom_panel: geometry collision box size=0.39 1 0.016; visual box size=0.39 1 0.016
- link wc_frame_left_side_panel: geometry collision box size=0.39 0.016 0.81; visual box size=0.39 0.016 0.81
- link wc_frame_right_side_panel: geometry collision box size=0.39 0.016 0.81; visual box size=0.39 0.016 0.81
- link wc_frame_top_panel: geometry collision box size=0.39 1 0.016; visual box size=0.39 1 0.016
Joints:
- added joint bc_frame_c1_v_shelf_joint: type fixed, parent bc_frame_base_link, child bc_frame_c1_v_shelf, origin xyz=0 -0.5 0.46
- added joint bc_frame_c2_v_shelf_joint: type fixed, parent bc_frame_base_link, child bc_frame_c2_v_shelf, origin xyz=0 -0.29999999999999993 0.46
- added joint bc_frame_c3_v_shelf_joint: type fixed, parent bc_frame_base_link, child bc_frame_c3_v_shelf, origin xyz=0 0.09999999999999998 0.46
- added joint bc_frame_h1_shelf_joint: type fixed, parent bc_frame_base_link, child bc_frame_h1_shelf, origin xyz=0 0.5000000000000001 0.6100000000000001
- added joint bc_frame_h2_shelf_joint: type fixed, parent bc_frame_base_link, child bc_frame_h2_shelf, origin xyz=0 0.5000000000000001 0.39000000000000007
- added joint wc_frame_c1_v_shelf_joint: type fixed, parent wc_frame_back_panel, child wc_frame_c1_v_shelf, origin xyz=0.187 0.09999999999999998 0
- added joint wc_frame_h1_shelf_joint: type fixed, parent wc_frame_back_panel, child wc_frame_h1_shelf, origin xyz=0.187 0 0.065
- added joint wc_frame_h2_shelf_joint: type fixed, parent wc_frame_back_panel, child wc_frame_h2_shelf, origin xyz=0.187 0 -0.135
- joint base_cabinet_c1_door_joint: origin xyz=0.3 -0.884 0.44 -> xyz=0.308 -0.9 0.46
- joint base_cabinet_c2_pull_out_front_panel_joint: origin xyz=0.308 -0.41600000000000004                        0.44 -> xyz=0.308                          -0.4                          0.46
- joint base_cabinet_c2_pull_out_handle_joint: origin xyz=0.008 0 0.34850000000000003 rpy=0 0 0 -> xyz=0.008 0 0.34800000000000003 rpy=0 0 0
- joint base_cabinet_c3_r1_drawer_front_panel_joint: origin xyz=0.308 -0.11599999999999999                      0.74 -> xyz=0.308                        -0.09999999999999998                        0.76
- joint base_cabinet_c3_r2_drawer_front_panel_joint: origin xyz=0.308 -0.11599999999999999                      0.54 -> xyz=0.308                        -0.09999999999999998                        0.56
- joint base_cabinet_c3_r3_drawer_front_panel_joint: origin xyz=0.308 -0.11599999999999999                      0.34 -> xyz=0.308                        -0.09999999999999998                        0.36000000000000004
- joint base_cabinet_c3_r4_drawer_front_panel_joint: origin xyz=0.308 -0.11599999999999999                      0.14 -> xyz=0.308                        -0.09999999999999998                        0.15999999999999992
- joint base_cabinet_c4_door_joint: origin xyz=0.3 0.08399999999999996 0.44 -> xyz=0.308                      0.09999999999999998                      0.46
- joint base_cabinet_c5_door_joint: origin xyz=0.3 0.884 0.44 -> xyz=0.308                      0.9                      0.46
- joint base_cabinet_reference: origin xyz=-2.7 0.2 0.04 rpy=0 0 0 -> xyz=-2.7 0.2 0.06 rpy=0 0 0
- joint bc_frame_back_panel_joint: origin xyz=-0.292 0 0.44 rpy=0 0 0 -> xyz=-0.292 0 0.46 rpy=0 0 0
- joint bc_frame_left_side_panel_joint: origin xyz=0 0.892 0.44 rpy=0 0 0 -> xyz=0 0.892 0.46 rpy=0 0 0
- joint bc_frame_right_side_panel_joint: origin xyz=0 -0.892 0.44 rpy=0 0 0 -> xyz=0 -0.892 0.46 rpy=0 0 0
- joint bc_frame_worktop_joint: origin xyz=0 0 0.8540000000000001 rpy=0 0 0 -> xyz=0 0 0.874
- joint wall_cabinet_c1_door_joint: origin xyz=0.366 -0.5 0 -> xyz=0.39 -0.5 0
- joint wall_cabinet_c2_door_joint: origin xyz=0.366 0.5 0 -> xyz=0.39 0.5 0
- joint wc_frame_bottom_panel_joint: origin xyz=0.179 0                    -0.397 rpy=0 0 0 -> xyz=0.187 0                    -0.397 rpy=0 0 0
- joint wc_frame_left_side_panel_joint: origin xyz=0.179                    0.492 0 rpy=0 0 0 -> xyz=0.187                    0.492 0 rpy=0 0 0
- joint wc_frame_right_side_panel_joint: origin xyz=0.179                    -0.492 0 rpy=0 0 0 -> xyz=0.187                    -0.492 0 rpy=0 0 0
- joint wc_frame_top_panel_joint: origin xyz=0.179 0                    0.397 rpy=0 0 0 -> xyz=0.187 0                    0.397 rpy=0 0 0

File: urdf/wall_cabinet.urdf (robot description, URDF)
Before this commit: robot wall_cabinet, 9 links, 8 joints
Links:
- added link wc_frame_c1_v_shelf, mass 10; collision box size=0.39 0.04 0.81; visual box size=0.39 0.04 0.81
- added link wc_frame_h1_shelf, mass 10; collision box size=0.39 1 0.02; visual box size=0.39 1 0.02
- added link wc_frame_h2_shelf, mass 10; collision box size=0.39 1 0.02; visual box size=0.39 1 0.02
- link wc_frame_bottom_panel: geometry collision box size=0.39 1 0.016; visual box size=0.39 1 0.016
- link wc_frame_left_side_panel: geometry collision box size=0.39 0.016 0.81; visual box size=0.39 0.016 0.81
- link wc_frame_right_side_panel: geometry collision box size=0.39 0.016 0.81; visual box size=0.39 0.016 0.81
- link wc_frame_top_panel: geometry collision box size=0.39 1 0.016; visual box size=0.39 1 0.016
Joints:
- added joint wc_frame_c1_v_shelf_joint: type fixed, parent wc_frame_back_panel, child wc_frame_c1_v_shelf, origin xyz=0.187 0.09999999999999998 0
- added joint wc_frame_h1_shelf_joint: type fixed, parent wc_frame_back_panel, child wc_frame_h1_shelf, origin xyz=0.187 0 0.065
- added joint wc_frame_h2_shelf_joint: type fixed, parent wc_frame_back_panel, child wc_frame_h2_shelf, origin xyz=0.187 0 -0.135
- joint wall_cabinet_c1_door_joint: origin xyz=0.366 -0.5 0 -> xyz=0.39 -0.5 0
- joint wall_cabinet_c2_door_joint: origin xyz=0.366 0.5 0 -> xyz=0.39 0.5 0
- joint wc_frame_bottom_panel_joint: origin xyz=0.179 0                    -0.397 rpy=0 0 0 -> xyz=0.187 0                    -0.397 rpy=0 0 0
- joint wc_frame_left_side_panel_joint: origin xyz=0.179                    0.492 0 rpy=0 0 0 -> xyz=0.187                    0.492 0 rpy=0 0 0
- joint wc_frame_right_side_panel_joint: origin xyz=0.179                    -0.492 0 rpy=0 0 0 -> xyz=0.187                    -0.492 0 rpy=0 0 0
- joint wc_frame_top_panel_joint: origin xyz=0.179 0                    0.397 rpy=0 0 0 -> xyz=0.187 0                    0.397 rpy=0 0 0

File: xacro/base_cabinet.xacro (robot description, xacro)
@@ -107,6 +107,6 @@
   <!-- Assembles -->
   <xacro:macro name="bc_frame">
-    <xacro:box_link prefix="bc_frame" link_name="base_link" mass="${bc_base_mass}" xdim="${bc_base_xdim}" ydim="${bc_base_ydim}"
-                    zdim="${bc_base_zdim}" material="White"/>
+    <xacro:box_link prefix="bc_frame" link_name="base_link" mass="${bc_base_mass}" xdim="${bc_base_xdim}"
+                    ydim="${bc_base_ydim}" zdim="${bc_base_zdim}" material="White"/>
     <xacro:box_link prefix="bc_frame" link_name="left_side_panel" mass="${bc_frame_side_panel_mass}"
                     xdim="${bc_frame_side_panel_xdim}" ydim="${bc_frame_side_panel_ydim}"
@@ -114,5 +114,6 @@
                     material="White"/>
     <joint name="bc_frame_left_side_panel_joint" type="fixed">
-      <origin xyz="0 ${(bc_base_ydim-bc_frame_side_panel_ydim)/2} ${(bc_base_zdim+bc_frame_side_panel_zdim)/2}" rpy="0 0 0"/>
+      <origin xyz="0 ${(bc_base_ydim-bc_frame_side_panel_ydim)/2} ${(bc_base_zdim+bc_frame_side_panel_zdim)/2}"
+              rpy="0 0 0"/>
       <parent link="bc_frame_base_link"/>
       <child link="bc_frame_left_side_panel"/>
@@ -123,5 +124,6 @@
                     material="White"/>
     <joint name="bc_frame_right_side_panel_joint" type="fixed">
-      <origin xyz="0 ${(-bc_base_ydim+bc_frame_side_panel_ydim)/2} ${(bc_base_zdim+bc_frame_side_panel_zdim)/2}" rpy="0 0 0"/>
+      <origin xyz="0 ${(-bc_base_ydim+bc_frame_side_panel_ydim)/2} ${(bc_base_zdim+bc_frame_side_panel_zdim)/2}"
+              rpy="0 0 0"/>
       <parent link="bc_frame_base_link"/>
       <child link="bc_frame_right_side_panel"/>
@@ -132,5 +134,6 @@
                     material="White"/>
     <joint name="bc_frame_back_panel_joint" type="fixed">
-      <origin xyz="${(-bc_base_xdim+bc_frame_back_panel_xdim)/2} 0 ${(bc_base_zdim+bc_frame_back_panel_zdim)/2}" rpy="0 0 0"/>
+      <origin xyz="${(-bc_base_xdim+bc_frame_back_panel_xdim)/2} 0 ${(bc_base_zdim+bc_frame_back_panel_zdim)/2}"
+              rpy="0 0 0"/>
       <parent link="bc_frame_base_link"/>
       <child link="bc_frame_back_panel"/>
@@ -140,7 +143,50 @@
                     material="White"/>
     <joint name="bc_frame_worktop_joint" type="fixed">
-      <origin xyz="0 0 ${(bc_base_zdim+worktop_zdim)/2+bc_frame_back_panel_zdim}" rpy="0 0 0"/>
+      <origin xyz="0 0 ${(bc_base_zdim+worktop_zdim)/2+bc_frame_zdim}"/>
       <parent link="bc_frame_base_link"/>
       <child link="bc_frame_worktop"/>
+    </joint>
+    <!-- Interior shelf -->
+    <!-- Vertical -->
+    <xacro:box_link prefix="bc_frame" link_name="c1_v_shelf" mass="${bc_v_shelf_mass}"
+                    xdim="${bc_v_shelf_xdim}" ydim="${bc_v_shelf_ydim}" zdim="${bc_v_shelf_zdim}"
+                    material="White"/>
+    <joint name="bc_frame_c1_v_shelf_joint" type="fixed">
+      <origin xyz="0 ${-bc_frame_ydim/2+bc_column_ydim} ${(bc_base_zdim+bc_frame_zdim)/2}"/>
+      <parent link="bc_frame_base_link"/>
+      <child link="bc_frame_c1_v_shelf"/>
+    </joint>
+    <xacro:box_link prefix="bc_frame" link_name="c2_v_shelf" mass="${bc_v_shelf_mass}"
+                    xdim="${bc_v_shelf_xdim}" ydim="${bc_v_shelf_ydim}" zdim="${bc_v_shelf_zdim}"
+                    material="White"/>
+    <joint name="bc_frame_c2_v_shelf_joint" type="fixed">
+      <origin xyz="0 ${-bc_frame_ydim/2+bc_column_ydim*1.5} ${(bc_base_zdim+bc_frame_zdim)/2}"/>
+      <parent link="bc_frame_base_link"/>
+      <child link="bc_frame_c2_v_shelf"/>
+    </joint>
+    <xacro:box_link prefix="bc_frame" link_name="c3_v_shelf" mass="${bc_v_shelf_mass}"
+                    xdim="${bc_v_shelf_xdim}" ydim="${bc_v_shelf_ydim}" zdim="${bc_v_shelf_zdim}"
+                    material="White"/>
+    <joint name="bc_frame_c3_v_shelf_joint" type="fixed">
+      <origin xyz="0 ${-bc_frame_ydim/2+bc_column_ydim*2.5} ${(bc_base_zdim+bc_frame_zdim)/2}"/>
+      <parent link="bc_frame_base_link"/>
+      <child link="bc_frame_c3_v_shelf"/>
+    </joint>
+    <!-- Horizontal -->
+    <xacro:box_link prefix="bc_frame" link_name="h1_shelf" mass="${bc_h_shelf_mass}"
+                    xdim="${bc_h_shelf_xdim}" ydim="${bc_h_shelf_ydim}" zdim="${bc_h_shelf_zdim}"
+                    material="White"/>
+    <joint name="bc_frame_h1_shelf_joint" type="fixed">
+      <origin xyz="0 ${-bc_frame_ydim/2+bc_column_ydim*3.5} ${(bc_base_zdim-bc_h_shelf_zdim)/2+bc_frame_zdim-0.24}"/>
+      <parent link="bc_frame_base_link"/>
+      <child link="bc_frame_h1_shelf"/>
+    </joint>
+    <xacro:box_link prefix="bc_frame" link_name="h2_shelf" mass="${bc_h_shelf_mass}"
+                    xdim="${bc_h_shelf_xdim}" ydim="${bc_h_shelf_ydim}" zdim="${bc_h_shelf_zdim}"
+                    material="White"/>
+    <joint name="bc_frame_h2_shelf_joint" type="fixed">
+      <origin xyz="0 ${-bc_frame_ydim/2+bc_column_ydim*3.5} ${(bc_base_zdim-bc_h_shelf_zdim)/2+bc_frame_zdim-0.46}"/>
+      <parent link="bc_frame_base_link"/>
+      <child link="bc_frame_h2_shelf"/>
     </joint>
   </xacro:macro>
@@ -157,32 +203,41 @@
     <!-- Rightmost 1st column -->
     <xacro:door prefix="${prefix}" name="c1_door" parent="bc_frame_base_link"
-                xyz="${bc_base_xdim/2} ${-bc_base_ydim/2+bc_frame_side_panel_ydim} ${(bc_base_zdim+bc_frame_side_panel_zdim)/2}"
+                xyz="${(bc_frame_xdim+bc_door_xdim)/2} ${-bc_frame_ydim/2} ${(bc_base_zdim+bc_frame_zdim)/2}"
                 mass="${bc_door_mass}" xdim="${bc_door_xdim}" ydim="${bc_door_ydim}" zdim="${bc_door_zdim}"
                 hinge="right" handle_xyz="0.008 0.35 0.28" handle_rpy="${M_PI/2} 0 0"/>
     <!-- Rightmost 2nd column -->
     <xacro:pull_out prefix="${prefix}" name="c2_pull_out" parent="bc_frame_base_link"
-                    xyz="${(bc_base_xdim+thickness)/2} ${bc_base_ydim/2-bc_frame_side_panel_ydim-bc_column_ydim*3.25}
-                       ${(bc_base_zdim+bc_frame_zdim)/2}"/>
+                    xyz="${(bc_frame_xdim+pull_out_front_panel_xdim)/2}
+                         ${-bc_frame_ydim/2+bc_column_ydim*1.25}
+                         ${(bc_base_zdim+bc_frame_zdim)/2}"/>
     <!-- Rightmost 3rd column -->
     <xacro:drawer prefix="${prefix}" name="c3_r1_drawer" parent="bc_frame_base_link"
-                  xyz="${(bc_base_xdim+drawer_front_panel_xdim)/2} ${bc_base_ydim/2-bc_frame_side_panel_ydim-bc_column_ydim*2.5}
-                     ${(bc_base_zdim-bc_row_zdim)/2+bc_frame_zdim}"/>
+                  xyz="${(bc_frame_xdim+drawer_front_panel_xdim)/2}
+                       ${-bc_frame_ydim/2+bc_column_ydim*2}
+                       ${(bc_base_zdim-bc_row_zdim)/2+bc_frame_zdim}"/>
     <xacro:drawer prefix="${prefix}" name="c3_r2_drawer" parent="bc_frame_base_link"
-                  xyz="${(bc_base_xdim+drawer_front_panel_xdim)/2} ${bc_base_ydim/2-bc_frame_side_panel_ydim-bc_column_ydim*2.5}
-                     ${(bc_base_zdim-bc_row_zdim*3)/2+bc_frame_zdim}"/>
+                  xyz="${(bc_frame_xdim+drawer_front_panel_xdim)/2}
+                       ${-bc_frame_ydim/2+bc_column_ydim*2}
+                       ${(bc_base_zdim-bc_row_zdim*3)/2+bc_frame_zdim}"/>
     <xacro:drawer prefix="${prefix}" name="c3_r3_drawer" parent="bc_frame_base_link"
-                  xyz="${(bc_base_xdim+drawer_front_panel_xdim)/2} ${bc_base_ydim/2-bc_frame_side_panel_ydim-bc_column_ydim*2.5}
-                     ${(bc_base_zdim-bc_row_zdim*5)/2+bc_frame_zdim}"/>
+                  xyz="${(bc_frame_xdim+drawer_front_panel_xdim)/2}
+                       ${-bc_frame_ydim/2+bc_column_ydim*2}
+                       ${(bc_base_zdim-bc_row_zdim*5)/2+bc_frame_zdim}"/>
     <xacro:drawer prefix="${prefix}" name="c3_r4_drawer" parent="bc_frame_base_link"
-                  xyz="${(bc_base_xdim+drawer_front_panel_xdim)/2} ${bc_base_ydim/2-bc_frame_side_panel_ydim-bc_column_ydim*2.5}
-                     ${(bc_base_zdim-bc_row_zdim*7)/2+bc_frame_zdim}"/>
+                  xyz="${(bc_frame_xdim+drawer_front_panel_xdim)/2}
+                       ${-bc_frame_ydim/2+bc_column_ydim*2}
+                       ${(bc_base_zdim-bc_row_zdim*7)/2+bc_frame_zdim}"/>
     <!-- Rightmost 4th column -->
     <xacro:door prefix="${prefix}" name="c4_door" parent="bc_frame_base_link"
-                xyz="${bc_base_xdim/2} ${bc_base_ydim/2-bc_frame_side_panel_ydim-bc_column_ydim*2} ${(bc_base_zdim+bc_frame_side_panel_zdim)/2}"
+                xyz="${(bc_frame_xdim+bc_door_xdim)/2}
+                     ${-bc_frame_ydim/2+bc_column_ydim*2.5}
+                     ${(bc_base_zdim+bc_frame_zdim)/2}"
                 mass="${bc_door_mass}" xdim="${bc_door_xdim}" ydim="${bc_door_ydim}" zdim="${bc_door_zdim}"
                 hinge="right" handle_xyz="0.008 0.35 0.28" handle_rpy="${M_PI/2} 0 0"/>
     <!-- Rightmost 5th column -->
     <xacro:door prefix="${prefix}" name="c5_door" parent="bc_frame_base_link"
-                xyz="${bc_base_xdim/2} ${bc_base_ydim/2-bc_frame_side_panel_ydim} ${(bc_base_zdim+bc_frame_side_panel_zdim)/2}"
+                xyz="${(bc_frame_xdim+bc_door_xdim)/2}
+                     ${-bc_frame_ydim/2+bc_column_ydim*4.5}
+                     ${(bc_base_zdim+bc_frame_zdim)/2}"
                 mass="${bc_door_mass}" xdim="${bc_door_xdim}" ydim="${bc_door_ydim}" zdim="${bc_door_zdim}"
                 hinge="left" handle_xyz="0.008 -0.35 0.28" handle_rpy="${M_PI/2} 0 0"/>
