Commit message: add interior shelf

File: xacro/include/components.xacro (robot description, xacro)
@@ -13,8 +13,8 @@
       <visual>
         <xacro:if value="${hinge == 'right'}">
-          <origin xyz="${xdim/2} ${ydim/2} 0"/>
+          <origin xyz="0 ${ydim/2} 0"/>
         </xacro:if>
         <xacro:if value="${hinge == 'left'}">
-          <origin xyz="${xdim/2} -${ydim/2} 0"/>
+          <origin xyz="0 ${-ydim/2} 0"/>
         </xacro:if>
         <xacro:if value="${hinge == 'none'}">
@@ -28,8 +28,8 @@
       <collision>
         <xacro:if value="${hinge == 'right'}">
-          <origin xyz="${xdim/2} ${ydim/2} 0"/>
+          <origin xyz="0 ${ydim/2} 0"/>
         </xacro:if>
         <xacro:if value="${hinge == 'left'}">
-          <origin xyz="${xdim/2} -${ydim/2} 0"/>
+          <origin xyz="0 ${-ydim/2} 0"/>
         </xacro:if>
         <xacro:if value="${hinge == 'none'}">
@@ -42,8 +42,8 @@
       <inertial>
         <xacro:if value="${hinge == 'right'}">
-          <origin xyz="${xdim/2} ${ydim/2} 0"/>
+          <origin xyz="0 ${ydim/2} 0"/>
         </xacro:if>
         <xacro:if value="${hinge == 'left'}">
-          <origin xyz="${xdim/2} -${ydim/2} 0"/>
+          <origin xyz="0 ${-ydim/2} 0"/>
         </xacro:if>
         <xacro:if value="${hinge == 'none'}">

File: xacro/include/materials.xacro (robot description, xacro)
@@ -13,5 +13,5 @@
     <color rgba="0.89 0.81 0.69 1.0"/>
   </material>
-  <material name="Green">
+  <material name="LightGreen">
     <color rgba="0.8 1 0.8 1.0"/>
   </material>

File: xacro/include/properties.xacro (robot description, xacro)
@@ -14,10 +14,12 @@
   <xacro:property name="wc_frame_ydim" value="1"/>
   <xacro:property name="wc_frame_zdim" value="0.81"/>
+  <!-- The wall cabinet has 2 columns, whose width are 0.6m and 0.4m, respectively -->
+  <xacro:property name="wc_column_ydim" value="0.6"/>
   <!-- https://www.ikea.com.hk/en/products/kitchen-cabinets-and-worktops/kitchen-cabinets/enhet-spr-49395118 -->
-  <xacro:property name="wc_frame_h_panel_xdim" value="${wc_frame_xdim-thickness}"/>
+  <xacro:property name="wc_frame_h_panel_xdim" value="${wc_frame_xdim}"/>
   <xacro:property name="wc_frame_h_panel_ydim" value="${wc_frame_ydim}"/>
   <xacro:property name="wc_frame_h_panel_zdim" value="${thickness}"/>
   <xacro:property name="wc_frame_h_panel_mass" value="20"/>
-  <xacro:property name="wc_frame_side_panel_xdim" value="${wc_frame_xdim-thickness}"/>
+  <xacro:property name="wc_frame_side_panel_xdim" value="${wc_frame_xdim}"/>
   <xacro:property name="wc_frame_side_panel_ydim" value="${thickness}"/>
   <xacro:property name="wc_frame_side_panel_zdim" value="${wc_frame_zdim}"/>
@@ -27,4 +29,13 @@
   <xacro:property name="wc_frame_back_panel_zdim" value="${wc_frame_zdim}"/>
   <xacro:property name="wc_frame_back_panel_mass" value="20"/>
+  <xacro:property name="wc_shelf_thickness" value="0.02"/>
+  <xacro:property name="wc_v_shelf_xdim" value="${wc_frame_xdim}"/>
+  <xacro:property name="wc_v_shelf_ydim" value="${wc_shelf_thickness*2}"/>
+  <xacro:property name="wc_v_shelf_zdim" value="${wc_frame_zdim}"/>
+  <xacro:property name="wc_v_shelf_mass" value="10"/>
+  <xacro:property name="wc_h_shelf_xdim" value="${wc_frame_xdim}"/>
+  <xacro:property name="wc_h_shelf_ydim" value="${wc_frame_ydim}"/>
+  <xacro:property name="wc_h_shelf_zdim" value="${wc_shelf_thickness}"/>
+  <xacro:property name="wc_h_shelf_mass" value="10"/>
   <!-- https://www.ikea.com.hk/en/products/kitchen-fronts/kitchen-fronts-cover-panels-and-plinth/enhet-art-90481556 -->
   <xacro:property name="wc_door_xdim" value="${thickness}"/>
@@ -34,5 +45,5 @@
   <xacro:property name="bc_base_xdim" value="0.6"/>
   <xacro:property name="bc_base_ydim" value="1.8"/>
-  <xacro:property name="bc_base_zdim" value="0.08"/>
+  <xacro:property name="bc_base_zdim" value="0.12"/>
   <xacro:property name="bc_base_mass" value="20"/>
   <!-- Frame refers to the main part of the cabinet -->
@@ -42,4 +53,13 @@
   <xacro:property name="bc_column_ydim" value="0.4"/>
   <xacro:property name="bc_row_zdim" value="${bc_frame_zdim/4}"/>
+  <xacro:property name="bc_shelf_thickness" value="0.02"/>
+  <xacro:property name="bc_v_shelf_xdim" value="${bc_frame_xdim}"/>
+  <xacro:property name="bc_v_shelf_ydim" value="${bc_shelf_thickness*2}"/>
+  <xacro:property name="bc_v_shelf_zdim" value="${bc_frame_zdim}"/>
+  <xacro:property name="bc_v_shelf_mass" value="10"/>
+  <xacro:property name="bc_h_shelf_xdim" value="${bc_frame_xdim}"/>
+  <xacro:property name="bc_h_shelf_ydim" value="${bc_column_ydim*2}"/>
+  <xacro:property name="bc_h_shelf_zdim" value="${bc_shelf_thickness}"/>
+  <xacro:property name="bc_h_shelf_mass" value="10"/>
   <xacro:property name="bc_frame_back_panel_xdim" value="${thickness}"/>
   <xacro:property name="bc_frame_back_panel_ydim" value="${bc_frame_ydim}"/>
@@ -68,5 +88,5 @@
   <!-- https://www.ikea.com.hk/en/products/kitchen-fixed-interiors/kitchen-fixed-interiors/maximera-art-70271111-->
   <xacro:property name="drawer_interior_xdim" value="0.542"/>
-  <xacro:property name="drawer_interior_ydim" value="0.364"/>
+  <xacro:property name="drawer_interior_ydim" value="0.35"/>
   <xacro:property name="drawer_interior_zdim" value="0.144"/>
   <xacro:property name="drawer_side_panel_xdim" value="${drawer_interior_xdim}"/>
@@ -84,6 +104,6 @@
   <!-- https://www.ikea.com.hk/en/products/kitchen-fronts/kitchen-fronts-cover-panels-and-plinth/askersund-art-50331776-->
   <xacro:property name="pull_out_front_panel_xdim" value="${thickness}"/>
-  <xacro:property name="pull_out_front_panel_ydim" value="0.197"/>
-  <xacro:property name="pull_out_front_panel_zdim" value="0.797"/>
+  <xacro:property name="pull_out_front_panel_ydim" value="${0.2-tolerance}"/>
+  <xacro:property name="pull_out_front_panel_zdim" value="${bc_frame_zdim-tolerance}"/>
   <xacro:property name="pull_out_front_panel_mass" value="1.66"/>
   <!-- https://www.ikea.com.hk/en/products/kitchen-fixed-interiors/kitchen-fixed-interiors/maximera-art-80297276-->

File: xacro/include/wall.xacro (robot description, xacro)
@@ -5,5 +5,5 @@
     <xacro:box_link prefix="lab" link_name="left_wall" mass="100"
                     xdim="${space_xdim}" ydim="${wall_thickness}" zdim="${space_zdim}"
-                    material="Green"/>
+                    material="LightGreen"/>
     <joint name="left_wall_joint" type="fixed">
       <origin xyz="0 ${(space_ydim+wall_thickness)/2} ${space_zdim/2}" rpy="0 0 0"/>
@@ -13,5 +13,5 @@
     <xacro:box_link prefix="lab" link_name="back_wall" mass="100"
                     xdim="${wall_thickness}" ydim="${space_ydim}" zdim="${space_zdim}"
-                    material="Green"/>
+                    material="LightGreen"/>
     <joint name="back_wall_joint" type="fixed">
       <origin xyz="${-(space_xdim+wall_thickness)/2} 0 ${space_zdim/2}" rpy="0 0 0"/>

File: xacro/wall_cabinet.xacro (robot description, xacro)
@@ -4,8 +4,10 @@
   <xacro:macro name="wc_frame">
     <xacro:box_link prefix="wc_frame" link_name="back_panel" mass="${wc_frame_back_panel_mass}"
-                    xdim="${wc_frame_back_panel_xdim}" ydim="${wc_frame_back_panel_ydim}" zdim="${wc_frame_back_panel_zdim}"
+                    xdim="${wc_frame_back_panel_xdim}" ydim="${wc_frame_back_panel_ydim}"
+                    zdim="${wc_frame_back_panel_zdim}"
                     material="White"/>
     <xacro:box_link prefix="wc_frame" link_name="left_side_panel" mass="${wc_frame_side_panel_mass}"
-                    xdim="${wc_frame_side_panel_xdim}" ydim="${wc_frame_side_panel_ydim}" zdim="${wc_frame_side_panel_zdim}"
+                    xdim="${wc_frame_side_panel_xdim}" ydim="${wc_frame_side_panel_ydim}"
+                    zdim="${wc_frame_side_panel_zdim}"
                     material="White"/>
     <joint name="wc_frame_left_side_panel_joint" type="fixed">
@@ -16,5 +18,6 @@
     </joint>
     <xacro:box_link prefix="wc_frame" link_name="right_side_panel" mass="${wc_frame_side_panel_mass}"
-                    xdim="${wc_frame_side_panel_xdim}" ydim="${wc_frame_side_panel_ydim}" zdim="${wc_frame_side_panel_zdim}"
+                    xdim="${wc_frame_side_panel_xdim}" ydim="${wc_frame_side_panel_ydim}"
+                    zdim="${wc_frame_side_panel_zdim}"
                     material="White"/>
     <joint name="wc_frame_right_side_panel_joint" type="fixed">
@@ -42,4 +45,31 @@
       <child link="wc_frame_bottom_panel"/>
     </joint>
+    <!-- Interior shelf -->
+    <!-- Vertical -->
+    <xacro:box_link prefix="wc_frame" link_name="c1_v_shelf" mass="${wc_v_shelf_mass}"
+                    xdim="${wc_v_shelf_xdim}" ydim="${wc_v_shelf_ydim}" zdim="${wc_v_shelf_zdim}"
+                    material="White"/>
+    <joint name="wc_frame_c1_v_shelf_joint" type="fixed">
+      <origin xyz="${(wc_frame_xdim-wc_frame_back_panel_xdim)/2} ${-wc_frame_ydim/2+wc_column_ydim} 0"/>
+      <parent link="wc_frame_back_panel"/>
+      <child link="wc_frame_c1_v_shelf"/>
+    </joint>
+    <!-- Horizontal -->
+    <xacro:box_link prefix="wc_frame" link_name="h1_shelf" mass="${wc_h_shelf_mass}"
+                    xdim="${wc_h_shelf_xdim}" ydim="${wc_h_shelf_ydim}" zdim="${wc_h_shelf_zdim}"
+                    material="White"/>
+    <joint name="wc_frame_h1_shelf_joint" type="fixed">
+      <origin xyz="${(wc_frame_xdim-wc_frame_back_panel_xdim)/2} 0 ${wc_frame_zdim/2-0.34}"/>
+      <parent link="wc_frame_back_panel"/>
+      <child link="wc_frame_h1_shelf"/>
+    </joint>
+    <xacro:box_link prefix="wc_frame" link_name="h2_shelf" mass="${wc_h_shelf_mass}"
+                    xdim="${wc_h_shelf_xdim}" ydim="${wc_h_shelf_ydim}" zdim="${wc_h_shelf_zdim}"
+                    material="White"/>
+    <joint name="wc_frame_h2_shelf_joint" type="fixed">
+      <origin xyz="${(wc_frame_xdim-wc_frame_back_panel_xdim)/2} 0 ${wc_frame_zdim/2-0.54}"/>
+      <parent link="wc_frame_back_panel"/>
+      <child link="wc_frame_h2_shelf"/>
+    </joint>
   </xacro:macro>
   <xacro:macro name="wall_cabinet" params="prefix connected_to:='' xyz:='0 0 0' rpy:='0 0 0'">
@@ -55,11 +85,12 @@
     <!-- Rightmost 1st column -->
     <xacro:door prefix="${prefix}" name="c1_door" parent="wc_frame_back_panel"
-                xyz="${wc_frame_side_panel_xdim-wc_door_xdim/2} ${-wc_frame_back_panel_ydim/2} 0"
-                mass="${door_mass}" xdim="${wc_door_xdim}" ydim="${0.6-tolerance}" zdim="${wc_door_zdim}"
+                xyz="${wc_frame_xdim-(wc_frame_back_panel_xdim-wc_door_xdim)/2} ${-wc_frame_back_panel_ydim/2} 0"
+                mass="${door_mass}" xdim="${wc_door_xdim}" ydim="${wc_column_ydim-tolerance}" zdim="${wc_door_zdim}"
                 hinge="right" handle_xyz="0.008 0.48 -0.35" handle_rpy="0 0 0"/>
     <!-- Rightmost 2nd column -->
     <xacro:door prefix="${prefix}" name="c2_door" parent="wc_frame_back_panel"
-                xyz="${wc_frame_side_panel_xdim-wc_door_xdim/2} ${wc_frame_back_panel_ydim/2} 0"
-                mass="${door_mass}" xdim="${wc_door_xdim}" ydim="${0.4-tolerance}" zdim="${wc_door_zdim}"
+                xyz="${wc_frame_xdim-(wc_frame_back_panel_xdim-wc_door_xdim)/2} ${wc_frame_back_panel_ydim/2} 0"
+                mass="${door_mass}" xdim="${wc_door_xdim}" ydim="${wc_frame_ydim-wc_column_ydim-tolerance}"
+                zdim="${wc_door_zdim}"
                 hinge="left" handle_xyz="0.008 -0.28 -0.35" handle_rpy="0 0 0"/>
   </xacro:macro>
