Commit message: add wall cabinet and urdf for the whole lab

File: xacro/wall_cabinet.xacro (robot description, xacro)
@@ -1,3 +1,90 @@
 <?xml version="1.0"?>
 <robot name="wall_cabinet" xmlns:xacro="http://wiki.ros.org/xacro">
+  <!-- Using meter, kg -->
+  <!-- Frame refers to the main part of the cabinet -->
+  <xacro:property name="wc_frame_xdim" value="0.39"/>
+  <xacro:property name="wc_frame_ydim" value="1"/>
+  <xacro:property name="wc_frame_zdim" value="0.81"/>
+  <xacro:property name="thickness" value="0.016"/>
+  <xacro:property name="tolerance" value="0.004"/>
+  <!-- https://www.ikea.com.hk/en/products/kitchen-cabinets-and-worktops/kitchen-cabinets/enhet-spr-49395118 -->
+  <xacro:property name="wc_frame_h_panel_xdim" value="${wc_frame_xdim-thickness}"/>
+  <xacro:property name="wc_frame_h_panel_ydim" value="${wc_frame_ydim}"/>
+  <xacro:property name="wc_frame_h_panel_zdim" value="${thickness}"/>
+  <xacro:property name="wc_frame_h_panel_mass" value="20"/>
+  <xacro:property name="wc_frame_side_panel_xdim" value="${wc_frame_xdim-thickness}"/>
+  <xacro:property name="wc_frame_side_panel_ydim" value="${thickness}"/>
+  <xacro:property name="wc_frame_side_panel_zdim" value="${wc_frame_zdim}"/>
+  <xacro:property name="wc_frame_side_panel_mass" value="10"/>
+  <xacro:property name="wc_frame_back_panel_xdim" value="${thickness}"/>
+  <xacro:property name="wc_frame_back_panel_ydim" value="${wc_frame_ydim}"/>
+  <xacro:property name="wc_frame_back_panel_zdim" value="${wc_frame_zdim}"/>
+  <xacro:property name="wc_frame_back_panel_mass" value="20"/>
+  <!-- https://www.ikea.com.hk/en/products/kitchen-fronts/kitchen-fronts-cover-panels-and-plinth/enhet-art-90481556 -->
+  <xacro:property name="door_xdim" value="${thickness}"/>
+  <xacro:property name="door_zdim" value="${wc_frame_zdim-tolerance}"/>
+  <xacro:property name="door_mass" value="3.31"/>
+  <!-- Assembles -->
+  <xacro:macro name="wc_frame">
+    <xacro:box_link prefix="wc_frame" link_name="back_panel" mass="${wc_frame_back_panel_mass}"
+                    xdim="${wc_frame_back_panel_xdim}" ydim="${wc_frame_back_panel_ydim}" zdim="${wc_frame_back_panel_zdim}"
+                    material="White"/>
+    <xacro:box_link prefix="wc_frame" link_name="left_side_panel" mass="${wc_frame_side_panel_mass}"
+                    xdim="${wc_frame_side_panel_xdim}" ydim="${wc_frame_side_panel_ydim}" zdim="${wc_frame_side_panel_zdim}"
+                    material="White"/>
+    <joint name="wc_frame_left_side_panel_joint" type="fixed">
+      <origin xyz="${(wc_frame_side_panel_xdim-wc_frame_back_panel_xdim)/2}
+                   ${(wc_frame_back_panel_ydim-wc_frame_side_panel_ydim)/2} 0" rpy="0 0 0"/>
+      <parent link="wc_frame_back_panel"/>
+      <child link="wc_frame_left_side_panel"/>
+    </joint>
+    <xacro:box_link prefix="wc_frame" link_name="right_side_panel" mass="${wc_frame_side_panel_mass}"
+                    xdim="${wc_frame_side_panel_xdim}" ydim="${wc_frame_side_panel_ydim}" zdim="${wc_frame_side_panel_zdim}"
+                    material="White"/>
+    <joint name="wc_frame_right_side_panel_joint" type="fixed">
+      <origin xyz="${(wc_frame_side_panel_xdim-wc_frame_back_panel_xdim)/2}
+                   ${(-wc_frame_back_panel_ydim+wc_frame_side_panel_ydim)/2} 0" rpy="0 0 0"/>
+      <parent link="wc_frame_back_panel"/>
+      <child link="wc_frame_right_side_panel"/>
+    </joint>
+    <xacro:box_link prefix="wc_frame" link_name="top_panel" mass="${wc_frame_h_panel_mass}"
+                    xdim="${wc_frame_h_panel_xdim}" ydim="${wc_frame_h_panel_ydim}" zdim="${wc_frame_h_panel_zdim}"
+                    material="White"/>
+    <joint name="wc_frame_top_panel_joint" type="fixed">
+      <origin xyz="${(wc_frame_h_panel_xdim-wc_frame_back_panel_xdim)/2} 0
+                   ${(wc_frame_back_panel_zdim-wc_frame_h_panel_zdim)/2}" rpy="0 0 0"/>
+      <parent link="wc_frame_back_panel"/>
+      <child link="wc_frame_top_panel"/>
+    </joint>
+    <xacro:box_link prefix="wc_frame" link_name="bottom_panel" mass="${wc_frame_h_panel_mass}"
+                    xdim="${wc_frame_h_panel_xdim}" ydim="${wc_frame_h_panel_ydim}" zdim="${wc_frame_h_panel_zdim}"
+                    material="White"/>
+    <joint name="wc_frame_bottom_panel_joint" type="fixed">
+      <origin xyz="${(wc_frame_h_panel_xdim-wc_frame_back_panel_xdim)/2} 0
+                   ${(-wc_frame_back_panel_zdim+wc_frame_h_panel_zdim)/2}" rpy="0 0 0"/>
+      <parent link="wc_frame_back_panel"/>
+      <child link="wc_frame_bottom_panel"/>
+    </joint>
+  </xacro:macro>
+  <xacro:macro name="wall_cabinet" params="prefix connected_to:='' xyz:='0 0 0' rpy:='0 0 0'">
+    <xacro:wc_frame/>
+    <xacro:unless value="${not connected_to}">
+      <joint name="${prefix}_${connected_to}_joint" type="fixed">
+        <parent link="${connected_to}"/>
+        <child link="wc_frame_back_panel"/>
+        <origin rpy="${rpy}" xyz="${xyz}"/>
+      </joint>
+    </xacro:unless>
+    <!-- The +x direction points from the back of the cabinet to the front -->
+    <!-- Rightmost 1st column -->
+    <xacro:door prefix="${prefix}" name="c1_door" parent="wc_frame_back_panel"
+                xyz="${wc_frame_side_panel_xdim-door_xdim/2} ${-wc_frame_back_panel_ydim/2} 0"
+                mass="${door_mass}" xdim="${door_xdim}" ydim="${0.6-tolerance}" zdim="${door_zdim}"
+                hinge="right"/>
+    <!-- Rightmost 2nd column -->
+    <xacro:door prefix="${prefix}" name="c2_door" parent="wc_frame_back_panel"
+                xyz="${wc_frame_side_panel_xdim-door_xdim/2} ${wc_frame_back_panel_ydim/2} 0"
+                mass="${door_mass}" xdim="${door_xdim}" ydim="${0.4-tolerance}" zdim="${door_zdim}"
+                hinge="left"/>
+  </xacro:macro>
 </robot>

Commit message: fixed

File: urdf/clover_lab.urdf (robot description, URDF)
Before this commit: robot clover_lab, 72 links, 71 joints
Joints:
- joint base_cabinet_c1_r1_drawer_front_panel_joint: origin xyz=0.3 -0.7                                 0.5800000000000001 -> xyz=0.02899999999999997 -0.7                                 0.5800000000000001
- joint base_cabinet_c1_r2_drawer_front_panel_joint: origin xyz=0.3 -0.7                                 0.33999999999999997 -> xyz=0.02899999999999997 -0.7                                 0.33999999999999997

File: xacro/base_cabinet.xacro (robot description, xacro)
@@ -150,5 +150,5 @@
                 hinge="right" handle_xyz="0.008 0.35 0.28" handle_rpy="${M_PI/2} 0 0"/>
     <xacro:drawer_interior prefix="${prefix}" name="c1_r1_drawer" parent="bc_frame_base_link"
-                           xyz="${bc_frame_xdim/2} ${(-bc_frame_ydim+bc_column_ydim)/2}
+                           xyz="${(bc_frame_xdim-c1_r1_drawer_interior_xdim)/2} ${(-bc_frame_ydim+bc_column_ydim)/2}
                                 ${bc_base_zdim+0.43+c1_r1_drawer_interior_zdim/2}"
                            xdim="${c1_r1_drawer_interior_xdim}" ydim="${c1_r1_drawer_interior_ydim}"
@@ -156,5 +156,5 @@
                            has_front_panel="true" has_side_panel="false" has_back_panel="false"/>
     <xacro:drawer_interior prefix="${prefix}" name="c1_r2_drawer" parent="bc_frame_base_link"
-                           xyz="${bc_frame_xdim/2} ${(-bc_frame_ydim+bc_column_ydim)/2}
+                           xyz="${(bc_frame_xdim-c1_r1_drawer_interior_xdim)/2} ${(-bc_frame_ydim+bc_column_ydim)/2}
                                 ${bc_base_zdim+0.12+c1_r2_drawer_interior_zdim/2}"
                            xdim="${c1_r2_drawer_interior_xdim}" ydim="${c1_r2_drawer_interior_ydim}"
