Commit message: major bug fixed

File: clover_lab_mujoco.urdf (robot description, URDF)
Before this commit: robot clover_lab, 72 links, 71 joints
Joints:
- joint base_cabinet_c1_r1_drawer_front_panel_joint: origin xyz=0.02899999999999997 -0.7                                 0.5800000000000001 -> xyz=0.292 -0.7                                 0.5800000000000001
- joint base_cabinet_c1_r2_drawer_front_panel_joint: origin xyz=0.02899999999999997 -0.7                                 0.33999999999999997 -> xyz=0.292 -0.7                                 0.33999999999999997

File: urdf/clover_lab.urdf (robot description, URDF)
Before this commit: robot clover_lab, 72 links, 71 joints
Joints:
- joint base_cabinet_c1_r1_drawer_front_panel_joint: origin xyz=0.02899999999999997 -0.7                                 0.5800000000000001 -> xyz=0.292 -0.7                                 0.5800000000000001
- joint base_cabinet_c1_r2_drawer_front_panel_joint: origin xyz=0.02899999999999997 -0.7                                 0.33999999999999997 -> xyz=0.292 -0.7                                 0.33999999999999997

File: xacro/base_cabinet.xacro (robot description, xacro)
@@ -150,5 +150,5 @@
                 hinge="right" handle_xyz="0.008 0.35 0.28" handle_rpy="${M_PI/2} 0 0"/>
     <xacro:drawer_interior prefix="${prefix}" name="c1_r1_drawer" parent="bc_frame_base_link"
-                           xyz="${(bc_frame_xdim-c1_r1_drawer_interior_xdim)/2} ${(-bc_frame_ydim+bc_column_ydim)/2}
+                           xyz="${(bc_frame_xdim-thickness)/2} ${(-bc_frame_ydim+bc_column_ydim)/2}
                                 ${bc_base_zdim+0.43+c1_r1_drawer_interior_zdim/2}"
                            xdim="${c1_r1_drawer_interior_xdim}" ydim="${c1_r1_drawer_interior_ydim}"
@@ -156,5 +156,5 @@
                            has_front_panel="true" has_side_panel="false" has_back_panel="false"/>
     <xacro:drawer_interior prefix="${prefix}" name="c1_r2_drawer" parent="bc_frame_base_link"
-                           xyz="${(bc_frame_xdim-c1_r1_drawer_interior_xdim)/2} ${(-bc_frame_ydim+bc_column_ydim)/2}
+                           xyz="${(bc_frame_xdim-thickness)/2} ${(-bc_frame_ydim+bc_column_ydim)/2}
                                 ${bc_base_zdim+0.12+c1_r2_drawer_interior_zdim/2}"
                            xdim="${c1_r2_drawer_interior_xdim}" ydim="${c1_r2_drawer_interior_ydim}"
